File: pcb/eprinter.kicad_sch (KiCad schematic)
At the start: 58 parts, among them J1 USB_C_Receptacle_USB2.0_16P, J2 AFC07-S24FCC-00, J3 Conn_01x02_Pin, Q1 Si2301, Q2 Si1308EDL, SW1 RESET, SW2 BOOT, U1 ESP32-C3-WROOM-02, U2 LM431BIM3X, U3 LM66100DCK, U4 MIC841HYC5, U5 XC6220B331MR

Commit message: Finalize JLCPCB order
Parts:
- C10, C16, C2: LCSC C77040 -> C19702
- C11, C12, C13, C14, C15, C17, C3, C9: LCSC C77046 -> C15849
- C4, C6: LCSC C77050 -> C14663
- D2: LCSC C83242 -> C2286
- J2: LCSC C720477 -> C11057
- R1: LCSC C2077177 -> C22936
- R10, R7: LCSC C844375 -> C23186
- R11, R2, R3, R6, R9: LCSC C169103 -> C25804
- R15: LCSC C313691 -> C22935
- R16: LCSC C2086340 -> C22939
- R4, R5: LCSC C71618 -> C23345
- R8: value 100 -> 470; LCSC C844724 -> C23179
- SW1: value RESET -> SW_PUSH
- SW2: value BOOT -> SW_PUSH
Other:
- moved on the sheet: D2, R8
Changed lines of the file:
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@@
 	(wire
 		(pts
-			(xy 88.9 132.08) (xy 93.98 132.08)
-		)
-		(stroke
-			(width 0)
-			(type default)
-		)
-	)
-	(wire
-		(pts
 			(xy 77.47 185.42) (xy 77.47 182.88)
 		)
@@
 	(wire
 		(pts
+			(xy 93.98 132.08) (xy 88.9 132.08)
+		)
+		(stroke
+			(width 0)
+			(type default)
+		)
+	)
+	(wire
+		(pts
 			(xy 115.57 91.44) (xy 115.57 93.98)
 		)
@@
 	(wire
 		(pts
+			(xy 93.98 133.35) (xy 93.98 132.08)
+		)
+		(stroke
+			(width 0)
+			(type default)
+		)
+	)
+	(wire
+		(pts
 			(xy 57.15 29.21) (xy 62.23 29.21)
 		)
@@
 			)
 		)
-		(property "LCSC" "C77040"
+		(property "LCSC" "C19702"
 			(at 234.95 30.48 0)
 			(hide yes)
@@
 			)
 		)
-		(property "LCSC" "C2077177"
+		(property "LCSC" "C22936"
 			(at 35.56 29.21 90)
 			(hide yes)
@@
 			)
 		)
-		(property "LCSC" "C77046"
+		(property "LCSC" "C15849"
 			(at 254 134.62 0)
 			(hide yes)
@@
 			)
 		)
-		(property "LCSC" "C169103"
+		(property "LCSC" "C25804"
 			(at 115.57 87.63 0)
 			(hide yes)
@@
 			)
 		)
-		(property "LCSC" "C77050"
+		(property "LCSC" "C14663"
 			(at 148.59 180.34 0)
 			(hide yes)
@@
 			)
 		)
-		(property "LCSC" "C169103"
+		(property "LCSC" "C25804"
 			(at 77.47 166.37 0)
 			(hide yes)
@@
 			)
 		)
-		(property "LCSC" "C77040"
+		(property "LCSC" "C19702"
 			(at 270.51 29.21 0)
 			(hide yes)
@@
 			)
 		)
-		(property "LCSC" "C77040"
+		(property "LCSC" "C19702"
 			(at 77.47 140.97 0)
 			(hide yes)
@@
 			)
 		)
-		(property "LCSC" "C71618"
+		(property "LCSC" "C23345"
 			(at 63.5 92.71 90)
 			(hide yes)
@@
 			)
 		)
-		(property "LCSC" "C844375"
+		(property "LCSC" "C23186"
 			(at 82.55 87.63 0)
 			(hide yes)
@@
 	(symbol
 		(lib_id "Device:LED")
-		(at 93.98 143.51 90)
+		(at 93.98 144.78 90)
 		(unit 1)
 		(body_style 1)
@@
 		(dnp no)
 		(property "Reference" "D2"
-			(at 88.392 141.986 90)
+			(at 88.392 143.256 90)
 			(show_name no)
 			(do_not_autoplace no)
@@
 		)
 		(property "Value" "LED"
-			(at 88.392 144.526 90)
+			(at 88.392 145.796 90)
 			(show_name no)
 			(do_not_autoplace no)
@@
 		)
 		(property "Footprint" "LED_SMD:LED_0603_1608Metric"
-			(at 93.98 143.51 0)
+			(at 93.98 144.78 0)
 			(hide yes)
 			(show_name no)
@@
 		)
 		(property "Datasheet" ""
-			(at 93.98 143.51 0)
+			(at 93.98 144.78 0)
 			(hide yes)
 			(show_name no)
@@
 		)
 		(property "Description" "Light emitting diode"
-			(at 93.98 143.51 0)
+			(at 93.98 144.78 0)
 			(hide yes)
 			(show_name no)
@@
 		)
 		(property "Sim.Pins" "1=K 2=A"
-			(at 93.98 143.51 0)
+			(at 93.98 144.78 0)
 			(hide yes)
 			(show_name no)
@@
 			)
 		)
-		(property "LCSC" "C83242"
-			(at 93.98 143.51 90)
+		(property "LCSC" "C2286"
+			(at 93.98 144.78 90)
 			(hide yes)
 			(show_name no)
@@
 			)
 		)
-		(property "LCSC" "C77046"
+		(property "LCSC" "C15849"
 			(at 237.49 97.79 0)
 			(hide yes)
@@
 			)
 		)
-		(property "LCSC" "C77046"
+		(property "LCSC" "C15849"
 			(at 224.79 144.78 0)
 			(hide yes)
@@
 			)
 		)
-		(property "LCSC" "C169103"
+		(property "LCSC" "C25804"
 			(at 48.26 34.29 0)
 			(hide yes)
@@
 			)
 		)
-		(property "LCSC" "C71618"
+		(property "LCSC" "C23345"
 			(at 63.5 87.63 90)
 			(hide yes)
@@
 			)
 		)
-		(property "LCSC" "C77046"
+		(property "LCSC" "C15849"
 			(at 245.11 139.7 0)
 			(hide yes)
@@
 			)
 		)
-		(property "LCSC" "C720477"
+		(property "LCSC" "C11057"
 			(at 207.01 113.03 0)
 			(hide yes)
@@
 			)
 		)
-		(property "LCSC" "C313691"
+		(property "LCSC" "C22935"
 			(at 144.78 121.92 0)
 			(hide yes)
@@
 			)
 		)
-		(property "LCSC" "C77046"
+		(property "LCSC" "C15849"
 			(at 234.95 142.24 0)
 			(hide yes)
@@
 			)
 		)
-		(property "LCSC" "C77050"
+		(property "LCSC" "C14663"
 			(at 119.38 180.34 0)
 			(hide yes)
@@
 			)
 		)
-		(property "Value" "RESET"
+		(property "Value" "SW_PUSH"
 			(at 64.77 180.34 90)
 			(show_name no)
@@
 	(symbol
 		(lib_id "Device:R")
-		(at 93.98 135.89 0)
+		(at 93.98 137.16 0)
 		(unit 1)
 		(body_style 1)
@@
 		(fields_autoplaced yes)
 		(property "Reference" "R8"
-			(at 96.52 134.6199 0)
+			(at 96.52 135.8899 0)
 			(show_name no)
 			(do_not_autoplace no)
@@
 			)
 		)
-		(property "Value" "100"
-			(at 96.52 137.1599 0)
+		(property "Value" "470"
+			(at 96.52 138.4299 0)
 			(show_name no)
 			(do_not_autoplace no)
@@
 		)
 		(property "Footprint" "Resistor_SMD:R_0603_1608Metric"
-			(at 92.202 135.89 90)
+			(at 92.202 137.16 90)
 			(hide yes)
 			(show_name no)
@@
 		)
 		(property "Datasheet" ""
-			(at 93.98 135.89 0)
+			(at 93.98 137.16 0)
 			(hide yes)
 			(show_name no)
@@
 		)
 		(property "Description" "Resistor"
-			(at 93.98 135.89 0)
+			(at 93.98 137.16 0)
 			(hide yes)
 			(show_name no)
@@
 			)
 		)
-		(property "LCSC" "C844724"
-			(at 93.98 135.89 0)
+		(property "LCSC" "C23179"
+			(at 93.98 137.16 0)
 			(hide yes)
 			(show_name no)
@@
 			)
 		)
-		(property "LCSC" "C169103"
+		(property "LCSC" "C25804"
 			(at 48.26 44.45 0)
 			(hide yes)
@@
 			)
 		)
-		(property "LCSC" "C169103"
+		(property "LCSC" "C25804"
 			(at 93.98 166.37 0)
 			(hide yes)
@@
 			)
 		)
-		(property "Value" "BOOT"
+		(property "Value" "SW_PUSH"
 			(at 95.25 180.34 90)
 			(show_name no)
@@
 			)
 		)
-		(property "LCSC" "C844375"
+		(property "LCSC" "C23186"
 			(at 95.25 87.63 0)
 			(hide yes)
@@
 			)
 		)
-		(property "LCSC" "C77046"
+		(property "LCSC" "C15849"
 			(at 274.32 121.92 0)
 			(hide yes)
@@
 			)
 		)
-		(property "LCSC" "C77046"
+		(property "LCSC" "C15849"
 			(at 262.89 129.54 0)
 			(hide yes)
@@
 	(symbol
 		(lib_id "power:GND")
-		(at 93.98 147.32 0)
+		(at 93.98 148.59 0)
 		(unit 1)
 		(body_style 1)
@@
 		(dnp no)
 		(property "Reference" "#PWR011"
-			(at 93.98 153.67 0)
+			(at 93.98 154.94 0)
 			(hide yes)
 			(show_name no)
@@
 		)
 		(property "Value" "GND"
-			(at 97.536 150.368 0)
+			(at 97.536 151.638 0)
 			(show_name no)
 			(do_not_autoplace no)
@@
 		)
 		(property "Footprint" ""
-			(at 93.98 147.32 0)
+			(at 93.98 148.59 0)
 			(hide yes)
 			(show_name no)
@@
 		)
 		(property "Datasheet" ""
-			(at 93.98 147.32 0)
+			(at 93.98 148.59 0)
 			(hide yes)
 			(show_name no)
@@
 		)
 		(property "Description" "Power symbol creates a global label with name \"GND\" , ground"
-			(at 93.98 147.32 0)
+			(at 93.98 148.59 0)
 			(hide yes)
 			(show_name no)
@@
 			)
 		)
-		(property "LCSC" "C2086340"
+		(property "LCSC" "C22939"
 			(at 154.94 125.73 0)
 			(hide yes)
@@
 			)
 		)
-		(property "LCSC" "C77046"
+		(property "LCSC" "C15849"
 			(at 77.47 179.07 0)
 			(hide yes)
