File: pcb/eprinter.kicad_sch (KiCad schematic)
At the start: 58 parts, among them J1 USB_C_Receptacle_USB2.0_16P, J2 AFC07-S24FCC-00, J3 Conn_01x02_Pin, Q1 Si2301, Q2 Si1308EDL, SW1 SW_PUSH, SW2 SW_PUSH, U1 ESP32-C3-WROOM-02, U2 LM431BIM3X, U3 LM66100DCK, U4 MIC841HYC5, U5 XC6220B331MR

Commit message: Refactor
Parts:
- removed C8: 4.7u, Capacitor_SMD:C_0603_1608Metric, symbol Device:C
- removed Q2: Si1308EDL, Package_TO_SOT_SMD:SOT-323_SC-70, symbol Transistor_FET:Si1308EDL
- removed R1: 1, Resistor_SMD:R_0603_1608Metric, symbol Device:R
- removed R16: 2.2, Resistor_SMD:R_0603_1608Metric, symbol Device:R
- removed R2, R3: 10k, Resistor_SMD:R_0603_1608Metric, symbol Device:R
- removed U2: LM431BIM3X, Package_TO_SOT_SMD:SOT-23, symbol eprinter:LM431BIM3X
- added C13: 1u, Capacitor_SMD:C_0603_1608Metric, symbol Device:C
- added Q2: BSS138, Package_TO_SOT_SMD:SOT-23, symbol Transistor_FET:BSS138
- added R13: 0.47, Resistor_SMD:R_0805_2012Metric, symbol Device:R
- added U2: LM3480-5.0, Package_TO_SOT_SMD:SOT-23, symbol Regulator_Linear:LM3480-5.0
- C10, C16, C2: footprint Capacitor_SMD:C_0603_1608Metric -> Capacitor_SMD:C_0805_2012Metric; LCSC C19702 -> C440198
- C17: value 1u -> 100n; LCSC C15849 -> C14663
- C5, C7: value 4.7u -> 10u; footprint Capacitor_SMD:C_0603_1608Metric -> Capacitor_SMD:C_0805_2012Metric; LCSC C90057 -> C440198
- L1: value 47uH/500mA -> 68uH/500mA; footprint eprinter:IND-SMD_L3.0-W3.0-1 -> eprinter:IND-SMD_L4.0-W4.0; LCSC C76865 -> (none)
- R10: renamed from R13; LCSC C123423 -> C23163
- R11: renamed from R14; value 1.2M -> 1M; LCSC C844338 -> C22935
- R12: renamed from R15; value 1M -> 10k; LCSC C22935 -> (none)
- R14: renamed from R17; LCSC C123423 -> C23163
- R15: renamed from R18; value 1.2M -> 1M; LCSC C844338 -> C22935
- R16: renamed from R19; value 2.4M -> 3M; LCSC C3008968 -> C23156
- R17: renamed from R20; value 360k -> 430k; LCSC C844159 -> C25969
- R18: renamed from R21; value 1.2M -> 1.5M; LCSC C844338 -> C4172
- R19: renamed from R22; LCSC C123423 -> C23163
- renumbered C12 to C11, C13 to C12, C9 to C8, C11 to C9, R4 to R1, R5 to R2, R6 to R3, R7 to R4, R8 to R5, R9 to R6, R10 to R7, R11 to R8, R12 to R9
Connections:
- net D_GDR: now also Q2.1 (G)
- net D_RESE: now also Q2.2 (S), R13.1
- net GND: now also C13.2, R13.2, U2.3 (GND)
- net SOLAR+: now also U2.2 (VI)
- net at D1.2 (A): now also U2.1 (VO)
- net at C7.2, D4.2 (A), L1.2: now also Q2.3 (D)
- net D_HLTCTL: now reaches J2.1 (Pin_1)
- net D_VGL: now reaches J2.4 (Pin_4)
- net D_VGL: now also C13.1
- net D_VSH2 renamed D_VGH
- no-connect marks 10 -> 9
Other:
- note added: "0.47 or 3 ohm depending on display"
- note added: "Solar+ and Vin are in 0 - 5.7V range divided to 0 - 1V. The ADC must be configured with 2.5dB attenuation covering 0 - 1.05V range."
- note added: "Vin < 5.5V Enable voltage: High Thresh = Vref(1.24V) * (R1 + R2 + R3) / R3 = 4.075V Low Thresh = Vref(1.24V) * (R1 + R2 + R3) / (R2 + R3) = 3.167V"
- note removed: "Solar+ and Vin are in 0 - 5.1V range divided to 0 - 1.04V. The ADC must be configured with 2.5dB attenuation covering 0 - 1.05V range."
- note removed: "Taken from GDEY042Z98 (4.2") datasheet TODO: see what components need to be changed for different sizes"
- note removed: "Vin < 5.5V Enable voltage: High Thresh = Vref(1.24V) * (R1 + R2 + R3) / R3 = 4.092V Low Thresh = Vref(1.24V) * (R1 + R2 + R3) / (R2 + R3) = 3.147V"
- moved on the sheet: C1, C10, C11, C12, C14, C15, C16, C17, C8, C9, D1, D3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

Commit message: Finish PCB v1
Parts:
- R10, R14, R19: LCSC C23163 -> C482196
- R16: value 3M -> 2M; LCSC C23156 -> C22976
- R17: value 430k -> 330k; LCSC C25969 -> C23137
- R18: value 1.5M -> 1M; LCSC C4172 -> C22935
Other:
- note added: "Vin < 5.5V Enable voltage: High Thresh = Vref(1.24V) * (R1 + R2 + R3) / R3 = 4.13V Low Thresh = Vref(1.24V) * (R1 + R2 + R3) / (R2 + R3) = 3.1V"
- note removed: "Vin < 5.5V Enable voltage: High Thresh = Vref(1.24V) * (R1 + R2 + R3) / R3 = 4.075V Low Thresh = Vref(1.24V) * (R1 + R2 + R3) / (R2 + R3) = 3.167V"
Changed lines of the file:
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@@
 		)
 	)
-	(text "Vin < 5.5V\nEnable voltage:\nHigh Thresh = Vref(1.24V) * (R1 + R2 + R3) / R3 = 4.075V\nLow Thresh = Vref(1.24V) * (R1 + R2 + R3) / (R2 + R3) = 3.167V"
+	(text "Vin < 5.5V\nEnable voltage:\nHigh Thresh = Vref(1.24V) * (R1 + R2 + R3) / R3 = 4.13V\nLow Thresh = Vref(1.24V) * (R1 + R2 + R3) / (R2 + R3) = 3.1V"
 		(exclude_from_sim no)
 		(at 200.914 17.78 0)
@@
 			)
 		)
-		(property "LCSC" "C23163"
+		(property "LCSC" "C482196"
 			(at 240.03 52.07 0)
 			(hide yes)
@@
 			)
 		)
-		(property "Value" "430k"
+		(property "Value" "330k"
 			(at 184.15 44.4499 0)
 			(show_name no)
@@
 			)
 		)
-		(property "LCSC" "C25969"
+		(property "LCSC" "C23137"
 			(at 181.61 43.18 0)
 			(hide yes)
@@
 			)
 		)
-		(property "Value" "3M"
+		(property "Value" "2M"
 			(at 184.15 33.0199 0)
 			(show_name no)
@@
 			)
 		)
-		(property "LCSC" "C23156"
+		(property "LCSC" "C22976"
 			(at 181.61 31.75 0)
 			(hide yes)
@@
 			)
 		)
-		(property "Value" "1.5M"
+		(property "Value" "1M"
 			(at 184.15 54.6099 0)
 			(show_name no)
@@
 			)
 		)
-		(property "LCSC" "C4172"
+		(property "LCSC" "C22935"
 			(at 181.61 53.34 0)
 			(hide yes)
@@
 			)
 		)
-		(property "LCSC" "C23163"
+		(property "LCSC" "C482196"
 			(at 132.08 166.37 0)
 			(hide yes)
@@
 			)
 		)
-		(property "LCSC" "C23163"
+		(property "LCSC" "C482196"
 			(at 161.29 166.37 0)
 			(hide yes)

Commit message: Switch to buck-boost converter to utilize more super cap capacity
Parts:
- removed U2: LM3480-5.0, Package_TO_SOT_SMD:SOT-23, symbol Regulator_Linear:LM3480-5.0
- removed U4: MIC841HYC5, Package_TO_SOT_SMD:SOT-353_SC-70-5, symbol eprinter:MIC841HYC5
- removed U5: XC6220B331MR, Package_TO_SOT_SMD:SOT-23-5, symbol Regulator_Linear:XC6220B331MR
- added L2: 0.47u, Inductor_SMD:L_1210_3225Metric, symbol Device:L
- added R20, R21: 510k, Resistor_SMD:R_0603_1608Metric, symbol Device:R
- added R22: 91k, Resistor_SMD:R_0603_1608Metric, symbol Device:R
- added R23: 4.7M, Resistor_SMD:R_0603_1608Metric, symbol Device:R
- added U2: TPS63802DLAR, eprinter:VSON-10_L3.0-W2.0-P0.50-TL, symbol eprinter:TPS63802DLAR
- added U6: ATL431BIDBZR, Package_TO_SOT_SMD:SOT-23-3, symbol Reference_Voltage:TL431DBZ
- C10: value 10u -> 22u; LCSC C440198 -> C45783
- R10, R14: LCSC C482196 -> C23163
- R13: footprint Resistor_SMD:R_0805_2012Metric -> Resistor_SMD:R_0603_1608Metric; LCSC (none) -> C23411; now fitted; now in the parts list
- R16: value 2M -> 1M; LCSC C22976 -> C22935
- R17: value 330k -> 680k; LCSC C23137 -> C25822
- R18: value 1M -> 4.7M; LCSC C22935 -> C23163
- R19: value 4.7M -> 510k; LCSC C482196 -> C23192
Connections:
- net +3V3: now also C10.1, R19.1, R23.2, U2.6 (VOUT); no longer C16.1
- net GND: now also R17.2, R21.2, R22.2, U2.2 (MODE), U2.3 (AGND), U2.8 (GND), U6.3 (A); no longer R18.2, R19.1
- net SOLAR+: now also D1.2 (A), R20.1, U6.1 (K)
- net VIN: now also C16.1, R18.1, U2.10 (VIN); no longer C10.1
- net at R19.2: now also R22.1, U2.4 (FB)
- net at R16.2, R17.1: now also R23.1, U2.1 (EN)
- new net: R18.2, U2.5 (PG)
- new net: L2.2, U2.7 (L2)
- new net: L2.1, U2.9 (L1)
- new net: R20.2, R21.1, U6.2 (REF)
Other:
- note added: "Vin < 5.5V Enable voltage: High Thresh = 2.95V Low Thresh = 1.98V"
- note removed: "Vin < 5.5V Enable voltage: High Thresh = Vref(1.24V) * (R1 + R2 + R3) / R3 = 4.13V Low Thresh = Vref(1.24V) * (R1 + R2 + R3) / (R2 + R3) = 3.1V"
- moved on the sheet: C1, D3, R9, U3
