File: pcb/eprinter.kicad_pcb (KiCad board)
At the start: 2 copper layers, 24.5 x 61 mm, 40 parts, among them J1 Conn_01x02_Pin, J2 Conn_01x08_Pin, J3 USB_C_Receptacle_USB2.0_16P, U1 MIC841HYC5, U2 XC6220B331MR, U3 ESP32-C3-WROOM-02

Commit message: Finish PCB routing
Parts:
- moved R2 4.55 mm to (155.2, 91.4)
- moved R3 4.55 mm to (153.7, 91.4)
- moved C2 0.84 mm to (157.5, 84.0)
- moved R10 0.84 mm to (161.5, 84.7)
- moved R9 0.84 mm to (159.5, 84.7)
Routing:
- net /SOLAR_V: track 0.00 -> 35.4 mm, vias 0 -> 2
- net /BAT_V: track 4.09 -> 38.1 mm, vias 0 -> 2
- net /SOLAR+: track 6.05 -> 30.8 mm, vias 0 -> 1
- net GND: track 4.23 -> 26.8 mm, vias 3 -> 53
- net +3V3: track 39.8 -> 53.5 mm, vias 0 -> 1
- net /D_MOSI: track 29.6 -> 41.9 mm, vias 0 -> 1
- net /D_SCK: track 24.9 -> 36.8 mm, vias 0 -> 1
- net Net-(J3-D--PadA7): track 36.2 -> 40.7 mm
- net Net-(J3-D+-PadA6): track 36.6 -> 41.1 mm
- net /USB_D-: track 12.5 -> 8.07 mm
- net /USB_D+: track 10.4 -> 5.95 mm
- net /D_RST: track 25.7 -> 28.3 mm, vias 2 -> 1
- net /D_DC: track 28.9 -> 31.4 mm, vias 2 -> 1
- net /D_CS: track 32.1 -> 34.6 mm, vias 2 -> 1
- net /D_BUSY: track 22.8 -> 24.6 mm, vias 2 -> 1
- added copper zone on In1.Cu, net GND
- added copper zone on In2.Cu, net GND
Other:
- copper layers 2 -> 4

Commit message: Refactor PCB
Parts:
- removed D4: 1N4733A, Diode_THT:D_DO-41_SOD81_P10.16mm_Horizontal
- removed the R4 at (159.5, 58.0)
- removed the U3 at (159.9, 101.4)
- added R2: 10k, Resistor_SMD:R_0603_1608Metric, F.Cu at (153.0, 58.0)
- added R3: 10k, Resistor_SMD:R_0603_1608Metric, F.Cu at (151.2, 58.0)
- added R6: 10k, Resistor_SMD:R_0603_1608Metric, F.Cu at (166.0, 60.8)
- added U1: TL431DBZ, Package_TO_SOT_SMD:SOT-23, F.Cu at (154.2, 62.0)
- added U4: ESP32-C3-WROOM-02, RF_Module:ESP32-C3-WROOM-02, F.Cu at (159.8, 101.4)
- added U5: LM66100DCK, Package_TO_SOT_SMD:SOT-363_SC-70-6, F.Cu at (162.5, 59.2)
- D1: value PMEG2010AEJ -> BAT54J
- moved R7 4.32 mm to (151.2, 52.2)
- moved TP2 4.26 mm to (153.2, 67.5)
- moved R9 4.19 mm to (168.2, 52.5)
- moved R1 3.79 mm to (154.2, 65.2)
- moved TP1 1.63 mm to (151.0, 60.5)
- moved D1 1.60 mm to (159.0, 62.5)
- moved R15 1.00 mm to (161.5, 67.5)
- moved R16 1.00 mm to (159.5, 67.5)
- moved R17 1.00 mm to (157.5, 67.5)
- moved D2 0.08 mm to (164.0, 62.8)
- renumbered R8 to R10, R9 to R11, R10 to R12, R11 to R13, R12 to R14, R13 to R15, R14 to R16, R15 to R17, R16 to R18, R17 to R19, R2 to R4, R3 to R5, R5 to R7, R6 to R8, R7 to R9, U1 to U2, U2 to U3
Connections:
- D2 pad 1: Net-(D1-K) -> Net-(D2-K)
- D2 pad 2: Net-(D2-A) -> /USB_5V
- R10 pad 1: Net-(D1-K) -> Net-(D2-K)
- TP3 pad 1: Net-(D1-K) -> Net-(D2-K)
Routing:
- net Net-(D2-K): track 0.00 -> 16.1 mm
- net Net-(D1-A): track 4.16 -> 15.1 mm
- net /USB_5V: track 10.8 -> 18.9 mm
- net GND: track 26.8 -> 34.1 mm, vias 53 -> 35
- net Net-(J3-CC1): track 7.92 -> 13.4 mm, vias 0 -> 2
- net Net-(J3-CC2): track 7.76 -> 12.3 mm
- net Net-(D2-A): track 4.36 -> 0.00 mm
- net Net-(U1-REF): track 0.00 -> 4.11 mm
- net /SOLAR+: track 30.8 -> 32.3 mm
- net Net-(D1-K): track 19.5 -> 21.0 mm, vias 0 -> 1
- net /VIN: track 25.6 -> 24.6 mm

Commit message: Finalize silk screen
Parts:
- removed TP1, TP2, TP3, TP4: TestPoint, TestPoint:TestPoint_Pad_1.0x1.0mm
Routing:
- net /SOLAR+: track 32.3 -> 28.9 mm
- net Net-(D1-A): track 15.1 -> 12.1 mm
- net /VIN: track 24.6 -> 22.2 mm
- net Net-(D2-K): track 16.1 -> 13.7 mm
Other:
- board text added: "ePrinter"
- board text added: "rev 0.1"

Commit message: Schematic verification
Parts:
- removed TP5, TP6: TestPoint, TestPoint:TestPoint_Pad_1.0x1.0mm
- added C10: 10u, Capacitor_SMD:C_0603_1608Metric, F.Cu at (121.3, 80.0)
- added C11: 1u, Capacitor_SMD:C_0603_1608Metric, F.Cu at (143.0, 105.5)
- added C12: 1u, Capacitor_SMD:C_0603_1608Metric, F.Cu at (143.0, 108.0)
- added C13: 1u, Capacitor_SMD:C_0603_1608Metric, F.Cu at (143.0, 110.5)
- added C14: 1u, Capacitor_SMD:C_0603_1608Metric, F.Cu at (143.0, 113.0)
- added C15: 1u, Capacitor_SMD:C_0603_1608Metric, F.Cu at (143.0, 115.5)
- added C16: 10u, Capacitor_SMD:C_0603_1608Metric, F.Cu at (119.3, 91.0)
- added C17: 1u, Capacitor_SMD:C_0603_1608Metric, F.Cu at (143.0, 120.5)
- added C8: 4.7u, Capacitor_SMD:C_0603_1608Metric, F.Cu at (130.1, 114.0)
- added C9: 1u, Capacitor_SMD:C_0603_1608Metric, F.Cu at (139.0, 120.5)
- added D4: MBR0530, Diode_SMD:D_SOD-123, F.Cu at (119.0, 104.2)
- added D5: MBR0530, Diode_SMD:D_SOD-123, F.Cu at (119.0, 107.6)
- added D6: MBR0530, Diode_SMD:D_SOD-123, F.Cu at (119.0, 111.0)
- added L1: 47uH/500mA, eprinter:IND-SMD_L3.0-W3.0-1, F.Cu at (125.7, 115.5)
- added Q1: Si2301, Package_TO_SOT_SMD:SOT-23, F.Cu at (124.3, 104.8)
- added Q2: Si1308EDL, Package_TO_SOT_SMD:SOT-323_SC-70, F.Cu at (118.1, 114.3)
- added R20: 360k, Resistor_SMD:R_0603_1608Metric, F.Cu at (117.0, 82.5)
- added R21: 1.2M, Resistor_SMD:R_0603_1608Metric, F.Cu at (117.0, 85.0)
- added R22: 4.7M, Resistor_SMD:R_0603_1608Metric, F.Cu at (117.0, 87.5)
- added SW1: SW_Push, eprinter:SW-SMD_L3.9-W3.0-P4.45, F.Cu at (130.0, 61.8)
- added SW2: SW_Push, eprinter:SW-SMD_L3.9-W3.0-P4.45, F.Cu at (136.0, 61.8)
- C2: value 100n -> 10u
- C3: value 100n -> 1u
- C4: value 1u -> 100n
- C5, C7: value 10u -> 4.7u
- C6: value 10u -> 100n
- D2: value PMEG2010AEJ -> LED; footprint Diode_SMD:D_SOD-323F -> LED_SMD:LED_0603_1608Metric
- D3: value LED -> PMEG2010AEJ; footprint LED_SMD:LED_0603_1608Metric -> Diode_SMD:D_SOD-323F
- J1: value Conn_01x02_Pin -> USB_C_Receptacle_USB2.0_16P; footprint Connector_PinHeader_2.54mm:PinHeader_1x02_P2.54mm_Vertical -> eprinter:USB-C_SMD-TYPE-C-31-M-12_1
- J2: value Conn_01x08_Pin -> Conn_01x26_Pin; footprint Connector_PinHeader_2.54mm:PinHeader_1x08_P2.54mm_Vertical -> eprinter:FPC-SMD_AFC07-S24FCC-00
- J3: value USB_C_Receptacle_USB2.0_16P -> Conn_01x02_Pin; footprint eprinter:USB-C_SMD-TYPE-C-31-M-12_1 -> Connector_PinHeader_2.54mm:PinHeader_1x02_P2.54mm_Vertical
- R10: value 0.1 -> 5.1k
- R11: value 4.7M -> 10k
- R12: value 1.2M -> 0.1
- R15: value 2.4M -> 1M
- R16: value 360k -> 2.2
- R17: value 1.2M -> 4.7M
- R18: value 10k -> 1.2M
- R19: value 4.7M -> 2.4M
- R9: value 5.1k -> 10k
- U1: value TL431DBZ -> ESP32-C3-WROOM-02; footprint Package_TO_SOT_SMD:SOT-23 -> RF_Module:ESP32-C3-WROOM-02
- U2: value MIC841HYC5 -> TL431DBZ; footprint Package_TO_SOT_SMD:SOT-353_SC-70-5 -> Package_TO_SOT_SMD:SOT-23
- U3: value XC6220B331MR -> LM66100DCK; footprint Package_TO_SOT_SMD:SOT-23-5 -> Package_TO_SOT_SMD:SOT-363_SC-70-6
- U4: value ESP32-C3-WROOM-02 -> MIC841HYC5; footprint RF_Module:ESP32-C3-WROOM-02 -> Package_TO_SOT_SMD:SOT-353_SC-70-5
- U5: value LM66100DCK -> XC6220B331MR; footprint Package_TO_SOT_SMD:SOT-363_SC-70-6 -> Package_TO_SOT_SMD:SOT-23-5
- moved J3 60.6 mm to (139.0, 109.0), turned to 0 degrees
- moved R8 57.7 mm to (112.5, 65.5), turned to 0 degrees
- moved R6 54.3 mm to (112.3, 69.0), turned to 0 degrees
- moved R16 54.0 mm to (134.7, 115.5), turned to 0 degrees
- moved R15 52.8 mm to (134.7, 113.0), turned to 0 degrees
- moved R13 52.2 mm to (116.3, 66.5), turned to 0 degrees
- moved R9 52.1 mm to (117.0, 62.0), turned to 0 degrees
- moved R14 49.6 mm to (116.3, 69.0), turned to 0 degrees
- moved R18 49.0 mm to (121.0, 64.5), turned to 0 degrees
- moved U5 48.8 mm to (122.0, 86.5)
- moved J2 48.6 mm to (160.0, 119.5)
- moved C3 47.7 mm to (125.2, 61.8), turned to 0 degrees
- moved C5 45.3 mm to (130.1, 106.5), turned to 0 degrees
- moved C4 43.8 mm to (125.2, 64.3), turned to 0 degrees
- moved D2 42.9 mm to (121.2, 59.2), turned to 0 degrees
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Connections:
- C2 pad 1: /SOLAR_V -> +3V3
- C3 pad 1: /BAT_V -> /CHIP_EN
- C4 pad 1: Net-(U4-EN) -> /SOLAR_V
- C5 pad 1: /VIN -> /D_3V3
- C6 pad 1: +3V3 -> /BAT_V
- C7 pad 1: +3V3 -> Net-(D5-K)
- C7 pad 2: GND -> Net-(D4-A)
- D2 pad 1: Net-(D2-K) -> GND
- D2 pad 2: /USB_5V -> Net-(D2-A)
- D3 pad 1: GND -> Net-(D3-K)
- D3 pad 2: Net-(D3-A) -> /USB_5V
- J1 pad 1: /SOLAR+ -> GND
- J2 pad 1: +3V3 -> unconnected-(J2-Pin_1-Pad1)
- J2 pad 2: GND -> /D_GDR
- J2 pad 3: /D_MOSI -> /D_RESE
- J2 pad 4: /D_SCK -> unconnected-(J2-Pin_4-Pad4)
- J2 pad 5: /D_CS -> /D_VSH2
- J2 pad 6: /D_DC -> /D_TSCL
- J2 pad 7: /D_RST -> /D_TSDA
- J2 pad 8: /D_BUSY -> GND
- J3 pad 1: GND -> /SOLAR+
- R10 pad 1: Net-(D2-K) -> Net-(J1-CC1)
- R10 pad 2: /VIN -> GND
- R11 pad 1: /SOLAR+ -> +3V3
- R11 pad 2: /SOLAR_V -> /D_EN
- R12 pad 1: /SOLAR_V -> Net-(D3-K)
- R12 pad 2: GND -> /VIN
- R13 pad 1: /VIN -> /SOLAR+
- R13 pad 2: /BAT_V -> /SOLAR_V
- R14 pad 1: /BAT_V -> /SOLAR_V
- R15 pad 1: /VIN -> /D_GDR
- R15 pad 2: Net-(U2-HTH) -> GND
- R16 pad 1: Net-(U2-HTH) -> /D_RESE
- R16 pad 2: Net-(U2-LTH) -> GND
- R17 pad 1: Net-(U2-LTH) -> /VIN
- R17 pad 2: GND -> /BAT_V
- R18 pad 1: +3V3 -> /BAT_V
- R18 pad 2: Net-(U4-EN) -> GND
- R19 pad 1: GND -> /VIN
- R19 pad 2: Net-(U2-OUT) -> Net-(U4-HTH)
- R2 pad 2: Net-(U1-REF) -> Net-(U2-REF)
- R3 pad 1: Net-(U1-REF) -> Net-(U2-REF)
- R4 pad 1: Net-(J3-D--PadA7) -> Net-(J1-D--PadA7)
- R5 pad 2: Net-(J3-D+-PadA6) -> Net-(J1-D+-PadA6)
- R6 pad 1: /USB_5V -> +3V3
- R6 pad 2: GND -> /CHIP_EN
- R7 pad 1: Net-(J3-CC2) -> Net-(J1-CC2)
- R8 pad 2: Net-(D3-A) -> Net-(D2-A)
- R9 pad 1: Net-(J3-CC1) -> +3V3
- R9 pad 2: GND -> /BOOT
- U1 pad 1: Net-(D1-A) -> +3V3
- U1 pad 2: Net-(U1-REF) -> /CHIP_EN
- U1 pad 3: GND -> /D_CS
- U2 pad 1: Net-(U2-HTH) -> Net-(D1-A)
- U2 pad 2: GND -> Net-(U2-REF)
- U2 pad 3: Net-(U2-LTH) -> GND
- U3 pad 1: /VIN -> Net-(D1-K)
- U3 pad 3: Net-(U2-OUT) -> Net-(D3-K)
- U3 pad 5: +3V3 -> unconnected-(U3-ST-Pad5)
- U4 pad 1: +3V3 -> Net-(U4-HTH)
- U4 pad 2: Net-(U4-EN) -> GND
- U4 pad 3: /D_CS -> Net-(U4-LTH)
- U4 pad 4: /D_DC -> Net-(U4-OUT)
- U4 pad 5: /D_RST -> /VIN
- U5 pad 1: Net-(D1-K) -> /VIN
- U5 pad 3: /USB_5V -> Net-(U4-OUT)
- U5 pad 5: GND -> +3V3
Routing:
- net +3V3: track 53.5 -> 0.00 mm, vias 1 -> 0
- net /D_MOSI: track 41.9 -> 0.00 mm, vias 1 -> 0
- net Net-(J3-D+-PadA6): track 41.1 -> 0.00 mm
- net Net-(J3-D--PadA7): track 40.7 -> 0.00 mm
- net /BAT_V: track 38.1 -> 0.00 mm, vias 2 -> 0
- net /D_SCK: track 36.8 -> 0.00 mm, vias 1 -> 0
- net /SOLAR_V: track 35.4 -> 0.00 mm, vias 2 -> 0
- net /D_CS: track 34.6 -> 0.00 mm, vias 1 -> 0
- net GND: track 34.1 -> 0.00 mm, vias 35 -> 0
- net /D_DC: track 31.4 -> 0.00 mm, vias 1 -> 0
- net /SOLAR+: track 28.9 -> 0.00 mm, vias 1 -> 0
- net /D_RST: track 28.3 -> 0.00 mm, vias 1 -> 0
- net /D_BUSY: track 24.6 -> 0.00 mm, vias 1 -> 0
- net /VIN: track 22.2 -> 0.00 mm
- net Net-(D1-K): track 21.0 -> 0.00 mm, vias 1 -> 0
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- removed copper zone on In1.Cu, net GND
- removed copper zone on In2.Cu, net GND
Other:
- board outline removed
- board text removed: "ePrinter"
- board text removed: "rev 0.1"

Commit message: Routing done
Parts:
- D3: value PMEG2010AEJ -> PMEG2010EJ
- J2: value Conn_01x26_Pin -> AFC07-S24FCC-00
- SW1: value SW_Push -> RESET
- SW2: value SW_Push -> BOOT
- U2: value TL431DBZ -> LM431BIM3X
- moved R17 53.9 mm to (164.3, 94.1), turned to -90 degrees
- moved R18 50.4 mm to (161.8, 94.1), turned to -90 degrees
- moved Q2 49.4 mm to (166.6, 105.0), turned to 90 degrees
- moved R22 48.0 mm to (165.0, 90.0), turned to 90 degrees
- moved C16 47.4 mm to (165.9, 82.3), turned to 90 degrees
- moved R14 45.1 mm to (153.8, 94.2), turned to -90 degrees
- moved R13 44.5 mm to (151.2, 94.2), turned to -90 degrees
- moved R21 44.3 mm to (161.0, 90.0), turned to -90 degrees
- moved R8 43.4 mm to (154.5, 76.3), turned to -90 degrees
- moved R6 43.3 mm to (155.5, 72.4), turned to -90 degrees
- moved C4 43.1 mm to (156.2, 94.2), turned to -90 degrees
- moved U5 42.4 mm to (164.4, 86.3)
- moved C10 42.2 mm to (163.4, 82.3), turned to 90 degrees
- moved C6 42.1 mm to (159.3, 94.1), turned to -90 degrees
- moved R20 42.0 mm to (158.4, 90.0), turned to 90 degrees
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Routing:
- net GND: track 0.00 -> 100.3 mm, vias 0 -> 24
- net +3V3: track 0.00 -> 95.0 mm
- net /D_DC: track 0.00 -> 77.9 mm, vias 0 -> 2
- net /D_EN: track 0.00 -> 77.5 mm, vias 0 -> 2
- net /D_BUSY: track 0.00 -> 75.9 mm, vias 0 -> 2
- net /D_CS: track 0.00 -> 73.6 mm, vias 0 -> 2
- net /D_RES: track 0.00 -> 71.9 mm, vias 0 -> 2
- net /D_SDA: track 0.00 -> 70.1 mm, vias 0 -> 2
- net /D_SCL: track 0.00 -> 64.5 mm, vias 0 -> 2
- net /SOLAR_V: track 0.00 -> 59.3 mm, vias 0 -> 2
- net /BAT_V: track 0.00 -> 55.0 mm, vias 0 -> 2
- net /CHIP_EN: track 0.00 -> 37.8 mm
- net /D_3V3: track 0.00 -> 30.6 mm, vias 0 -> 2
- net /VIN: track 0.00 -> 24.8 mm
- net Net-(D1-K): track 0.00 -> 23.4 mm
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- added copper zone on In1.Cu, net GND
- added copper zone on In2.Cu, net GND
Other:
- board outline added: 28 x 70 mm

Commit message: PCB silkscreen done and LCSC part selection
Routing:
- net /SOLAR+: track 7.93 -> 9.65 mm
Other:
- board text added: "+"
- board text added: "5F/5.5V"
- board text added: "BOOT"
- board text added: "RST"
- board text added: "ePrinter"

Commit message: Finalize JLCPCB order
Parts:
- R8: value 100 -> 470
- SW1: value RESET -> SW_PUSH
- SW2: value BOOT -> SW_PUSH
Changed lines of the file:
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@@
 			(layer "F.SilkS"
 				(type "Top Silk Screen")
-				(color "Black")
 			)
 			(layer "F.Paste"
@@
 			(layer "F.Mask"
 				(type "Top Solder Mask")
-				(color "White")
 				(thickness 0.01)
 			)
@@
 			(layer "B.Mask"
 				(type "Bottom Solder Mask")
-				(color "White")
 				(thickness 0.01)
 			)
@@
 			(layer "B.SilkS"
 				(type "Bottom Silk Screen")
-				(color "Black")
 			)
 			(copper_finish "None")
@@
 			)
 		)
-		(property "LCSC" ""
+		(property "LCSC" "C844338"
 			(at 0 0 270)
 			(unlocked yes)
@@
 			)
 		)
-		(property "LCSC" ""
+		(property "LCSC" "C23186"
 			(at 0 0 270)
 			(unlocked yes)
@@
 			)
 		)
-		(property "LCSC" ""
+		(property "LCSC" "C23345"
 			(at 0 0 90)
 			(unlocked yes)
@@
 			)
 		)
-		(property "LCSC" ""
+		(property "LCSC" "C14663"
 			(at 0 0 270)
 			(unlocked yes)
@@
 			)
 		)
-		(property "LCSC" ""
+		(property "LCSC" "C23186"
 			(at 0 0 90)
 			(unlocked yes)
@@
 			)
 		)
-		(property "LCSC" ""
+		(property "LCSC" "C2286"
 			(at 0 0 270)
 			(unlocked yes)
@@
 			)
 		)
-		(property "LCSC" ""
+		(property "LCSC" "C123423"
 			(at 0 0 270)
 			(unlocked yes)
@@
 			)
 		)
-		(property "LCSC" ""
+		(property "LCSC" "C25804"
 			(at 0 0 270)
 			(unlocked yes)
@@
 			)
 		)
-		(property "LCSC" ""
+		(property "LCSC" "C15849"
 			(at 0 0 90)
 			(unlocked yes)
@@
 			)
 		)
-		(property "LCSC" ""
+		(property "LCSC" "C25804"
 			(at 0 0 270)
 			(unlocked yes)
@@
 			)
 		)
-		(property "LCSC" ""
+		(property "LCSC" "C15849"
 			(at 0 0 90)
 			(unlocked yes)
@@
 			)
 		)
-		(property "LCSC" ""
+		(property "LCSC" "C15849"
 			(at 0 0 90)
 			(unlocked yes)
@@
 			)
 		)
-		(property "LCSC" ""
+		(property "LCSC" "C22935"
 			(at 0 0 90)
 			(unlocked yes)
@@
 			)
 		)
-		(property "LCSC" ""
+		(property "LCSC" "C123423"
 			(at 0 0 270)
 			(unlocked yes)
@@
 			)
 		)
-		(property "LCSC" ""
+		(property "LCSC" "C19702"
 			(at 0 0 270)
 			(unlocked yes)
@@
 			)
 		)
-		(property "LCSC" ""
+		(property "LCSC" "C23345"
 			(at 0 0 270)
 			(unlocked yes)
@@
 			)
 		)
-		(property "LCSC" ""
+		(property "LCSC" "C22939"
 			(at 0 0 270)
 			(unlocked yes)
@@
 			)
 		)
-		(property "LCSC" ""
+		(property "LCSC" "C15849"
 			(at 0 0 90)
 			(unlocked yes)
@@
 			)
 		)
-		(property "LCSC" ""
+		(property "LCSC" "C25804"
 			(at 0 0 270)
 			(unlocked yes)
@@
 			)
 		)
-		(property "Value" "BOOT"
+		(property "Value" "SW_PUSH"
 			(at 0 3.541199 90)
 			(layer "F.Fab")
@@
 			)
 		)
-		(property "LCSC" ""
+		(property "LCSC" "C25804"
 			(at 0 0 270)
 			(unlocked yes)
@@
 			)
 		)
-		(property "LCSC" ""
+		(property "LCSC" "C3008968"
 			(at 0 0 270)
 			(unlocked yes)
@@
 			)
 		)
-		(property "LCSC" ""
+		(property "LCSC" "C844273"
 			(at 0 0 270)
 			(unlocked yes)
@@
 			)
 		)
-		(property "LCSC" ""
+		(property "LCSC" "C90057"
 			(at 0 0 90)
 			(unlocked yes)
@@
 			)
 		)
-		(property "LCSC" ""
+		(property "LCSC" "C25804"
 			(at 0 0 270)
 			(unlocked yes)
@@
 		(sheetname "/")
 		(sheetfile "eprinter.kicad_sch")
-		(attr smd exclude_from_bom)
+		(units
+			(unit
+				(name "A")
+				(pins "1" "2")
+			)
+		)
+		(attr smd exclude_from_pos_files exclude_from_bom dnp)
 		(duplicate_pad_numbers_are_jumpers no)
 		(fp_line
@@
 			)
 		)
-		(property "LCSC" "C720477"
+		(property "LCSC" "C11057"
 			(at 0 0 0)
 			(unlocked yes)
@@
 			)
 		)
-		(property "Value" "100"
+		(property "Value" "470"
 			(at 0 1.43 90)
 			(layer "F.Fab")
@@
 			)
 		)
-		(property "LCSC" ""
+		(property "LCSC" "C23179"
 			(at 0 0 270)
 			(unlocked yes)
@@
 			)
 		)
-		(property "Value" "RESET"
+		(property "Value" "SW_PUSH"
 			(at 0 3.541199 90)
 			(layer "F.Fab")
@@
 			)
 		)
-		(property "LCSC" ""
+		(property "LCSC" "C14663"
 			(at 0 0 270)
 			(unlocked yes)
@@
 			)
 		)
-		(attr through_hole exclude_from_bom)
+		(attr through_hole exclude_from_pos_files exclude_from_bom dnp)
 		(duplicate_pad_numbers_are_jumpers no)
 		(fp_line
@@
 		(sheetname "/")
 		(sheetfile "eprinter.kicad_sch")
+		(units
+			(unit
+				(name "A")
+				(pins "2" "18" "17" "16" "15" "3" "4" "5" "6" "7" "8" "10" "13" "14"
+					"1" "9" "19" "11" "12"
+				)
+			)
+		)
 		(attr smd)
 		(duplicate_pad_numbers_are_jumpers no)
@@
 			)
 		)
-		(property "LCSC" ""
+		(property "LCSC" "C844338"
 			(at 0 0 270)
 			(unlocked yes)
@@
 			)
 		)
-		(property "LCSC" ""
+		(property "LCSC" "C15849"
 			(at 0 0 90)
 			(unlocked yes)
@@
 			)
 		)
-		(property "LCSC" ""
+		(property "LCSC" "C844338"
 			(at 0 0 270)
 			(unlocked yes)
@@
 			)
 		)
-		(property "LCSC" ""
+		(property "LCSC" "C15849"
 			(at 0 0 90)
 			(unlocked yes)
@@
 			)
 		)
-		(property "LCSC" ""
+		(property "LCSC" "C123423"
 			(at 0 0 90)
 			(unlocked yes)
@@
 			)
 		)
-		(property "LCSC" ""
+		(property "LCSC" "C22936"
 			(at 0 0 0)
 			(unlocked yes)
@@
 			)
 		)
-		(property "LCSC" ""
+		(property "LCSC" "C844159"
 			(at 0 0 90)
 			(unlocked yes)
@@
 			)
 		)
-		(property "LCSC" ""
+		(property "LCSC" "C90057"
 			(at 0 0 90)
 			(unlocked yes)
@@
 			)
 		)
-		(property "LCSC" ""
+		(property "LCSC" "C19702"
 			(at 0 0 90)
 			(unlocked yes)
@@
 			)
 		)
-		(property "LCSC" ""
+		(property "LCSC" "C15849"
 			(at 0 0 90)
 			(unlocked yes)
@@
 			)
 		)
-		(property "LCSC" ""
+		(property "LCSC" "C90057"
 			(at 0 0 0)
 			(unlocked yes)
@@
 			)
 		)
-		(property "LCSC" ""
+		(property "LCSC" "C15849"
 			(at 0 0 90)
 			(unlocked yes)
@@
 			)
 		)
-		(property "LCSC" ""
+		(property "LCSC" "C19702"
 			(at 0 0 90)
 			(unlocked yes)

Commit message: Refactor
Parts:
- removed the C8 at (156.8, 104.9)
- removed the R1 at (152.5, 88.5)
- removed the R15 at (163.8, 104.9)
- removed the R16 at (166.8, 108.9)
- removed the R2 at (155.0, 85.0)
- removed the R3 at (152.5, 85.0)
- added C13: 1u, Capacitor_SMD:C_0603_1608Metric, F.Cu at (166.2, 108.9)
- added R12: 10k, Resistor_SMD:R_0603_1608Metric, F.Cu at (169.4, 107.8)
- added R13: 0.47, Resistor_SMD:R_0805_2012Metric, F.Cu at (169.4, 105.0)
- C10, C16, C2: footprint Capacitor_SMD:C_0603_1608Metric -> Capacitor_SMD:C_0805_2012Metric
- C17: value 1u -> 100n
- C5, C7: value 4.7u -> 10u; footprint Capacitor_SMD:C_0603_1608Metric -> Capacitor_SMD:C_0805_2012Metric
- L1: value 47uH/500mA -> 68uH/500mA; footprint eprinter:IND-SMD_L3.0-W3.0-1 -> eprinter:IND-SMD_L4.0-W4.0
- Q2: value Si1308EDL -> BSS138; footprint Package_TO_SOT_SMD:SOT-323_SC-70 -> Package_TO_SOT_SMD:SOT-23
- R11: renamed from R14; value 1.2M -> 1M
- R15: renamed from R18; value 1.2M -> 1M
- R16: renamed from R19; value 2.4M -> 3M
- R17: renamed from R20; value 360k -> 430k
- R18: renamed from R21; value 1.2M -> 1.5M
- U2: value LM431BIM3X -> LM3480-5.0
- moved U2 5.27 mm to (153.6, 85.9)
- moved D1 3.01 mm to (154.5, 81.0)
- moved R9 2.81 mm to (158.1, 81.9)
- moved R19 2.50 mm to (162.5, 90.0)
- moved Q2 1.89 mm to (165.0, 104.0), turned to 0 degrees
- moved C7 1.62 mm to (156.8, 103.5), turned to 90 degrees
- moved R16 1.50 mm to (154.5, 90.0)
- moved R17 1.50 mm to (156.9, 90.0)
- moved R18 1.50 mm to (159.5, 90.0)
- moved C4 1.29 mm to (157.5, 93.8)
- moved R10 1.29 mm to (152.5, 93.8)
- moved R11 1.29 mm to (155.0, 93.8)
- moved C6 1.29 mm to (160.5, 93.8)
- moved R14 1.29 mm to (165.5, 93.8)
- moved R15 1.29 mm to (163.0, 93.8)
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- renumbered C12 to C11, C13 to C12, C9 to C8, C11 to C9, R4 to R1, R13 to R10, R17 to R14, R22 to R19, R5 to R2, R6 to R3, R7 to R4, R8 to R5, R9 to R6, R10 to R7, R11 to R8, R12 to R9
Connections:
- net /D_VSH2 renamed /D_VGH
- J2 pad 1: unconnected-(J2-Pin_1-Pad1) -> /D_HLTCTL
- J2 pad 4: unconnected-(J2-Pin_4-Pad4) -> /D_VGL
- U2 pad 2: Net-(U2-REF) -> /SOLAR+
Routing:
- net GND: track 100.3 -> 86.3 mm, vias 24 -> 30
- net Net-(D1-A): track 14.0 -> 2.90 mm
- net Net-(U2-REF): track 7.84 -> 0.00 mm
- net /D_RESE: track 8.61 -> 14.4 mm
- net /D_3V3: track 30.6 -> 35.6 mm
- net /D_VGL: track 0.00 -> 4.86 mm
- net /SOLAR+: track 9.65 -> 13.1 mm
- net Net-(D3-K): track 11.3 -> 14.1 mm
- net Net-(D1-K): track 23.4 -> 20.9 mm
- net /D_GDR: track 16.2 -> 18.2 mm
- net /D_PREVGH: track 12.3 -> 10.5 mm
- net /SOLAR_V: track 59.3 -> 57.7 mm
- net Net-(D5-K): track 5.87 -> 7.42 mm
- net /BAT_V: track 55.0 -> 54.5 mm
Other:
- board text added: "v1"
